Commit message: meshes folder

File: src/matrice100/urdf/m100.urdf (robot description, URDF)
Before this commit: robot m100, 5 links, 4 joints
Links:
- link base_link: geometry visual mesh filename=package://matrice100/mesh/met.STL scale=4 4 4
- link leg1: geometry visual mesh filename=package://matrice100/mesh/leg1.STL scale=4 4 4
- link leg2: geometry visual mesh filename=package://matrice100/mesh/leg1.STL scale=4 4 4
- link leg3: geometry visual mesh filename=package://matrice100/mesh/leg1.STL scale=4 4 4
- link leg4: geometry visual mesh filename=package://matrice100/mesh/leg1.STL scale=4 4 4

Commit message: colors and rotating props

File: src/matrice100/urdf/m100.urdf (robot description, URDF)
Before this commit: robot m100, 5 links, 4 joints
Links:
- added link prop1; visual box size=0.8 0.1 0.05
- added link prop2; visual box size=0.8 0.1 0.05
- added link prop3; visual box size=0.8 0.1 0.05
- added link prop4; visual box size=0.8 0.1 0.05
Joints:
- added joint prop1: type continuous, parent leg1, child prop1, origin xyz=0.92 -0.92 0.87, axis 0 0 1
- added joint prop2: type continuous, parent leg2, child prop2, origin xyz=0.92 0.92 0.87, axis 0 0 1
- added joint prop3: type continuous, parent leg3, child prop3, origin xyz=-0.92 0.92 0.87, axis 0 0 1
- added joint prop4: type continuous, parent leg4, child prop4, origin xyz=-0.92 -0.92 0.87, axis 0 0 1
